Commit message: Update files

File: freehicle_description/urdf/freehicle/freehicle.xacro (robot description, xacro)
@@ -1,3 +1,90 @@
 <?xml version="1.0" ?>
 <robot name="hivebot" xmlns:xacro="http://www.ros.org/wiki/xacro">
+    <xacro:property name="TUBE_RADIUS" value="8e-3"/>
+    <xacro:property name="CENTER_TUBE_LENGTH" value="0.8382"/>
+    <xacro:property name="FRONT_TUBE_LENGTH" value="0.4826"/>
+    <xacro:property name="BACK_TUBE_LENGTH" value="0.28"/>
+    <xacro:property name="PI" value="3.1415926"/>
+    <xacro:include filename="$(find freehicle_description)/urdf/freehicle/wheel.xacro" />
+    <link name="body">
+        <inertial>
+            <mass value="30"/>
+            <origin rpy="0 0 0" xyz="0 0 0"/>
+            <inertia ixx="1" ixy="0.0" ixz="0.0"
+                     iyy="1" iyz="0.0"
+                     izz="1"/>
+        </inertial>
+        <collision name="center_tube">
+            <origin rpy="0 ${PI/2} 0" xyz="0 0 0"/>
+            <geometry>
+                <cylinder radius="${TUBE_RADIUS}" length="${CENTER_TUBE_LENGTH}" />
+            </geometry>
+        </collision>
+        <visual name="center_tube">
+            <origin rpy="0 ${PI/2} 0" xyz="0 0 0"/>
+            <geometry>
+                <cylinder radius="${TUBE_RADIUS}" length="${CENTER_TUBE_LENGTH}" />
+            </geometry>
+        </visual>
+        <collision name="back_tube">
+            <origin rpy="${PI/2} 0 0" xyz="${CENTER_TUBE_LENGTH/2} 0 0"/>
+            <geometry>
+                <cylinder radius="${TUBE_RADIUS}" length="${FRONT_TUBE_LENGTH}" />
+            </geometry>
+        </collision>
+        <visual name="back_tube">
+            <origin rpy="${PI/2} 0 0" xyz="${CENTER_TUBE_LENGTH/2} 0 0"/>
+            <geometry>
+                <cylinder radius="${TUBE_RADIUS}" length="${FRONT_TUBE_LENGTH}" />
+            </geometry>
+        </visual>
+        <collision name="back_tube">
+            <origin rpy="${PI/2} 0 0" xyz="-${CENTER_TUBE_LENGTH/2} 0 0"/>
+            <geometry>
+                <cylinder radius="${TUBE_RADIUS}" length="${BACK_TUBE_LENGTH}" />
+            </geometry>
+        </collision>
+        <visual name="back_tube">
+            <origin rpy="${PI/2} 0 0" xyz="-${CENTER_TUBE_LENGTH/2} 0 0"/>
+            <geometry>
+                <cylinder radius="${TUBE_RADIUS}" length="${BACK_TUBE_LENGTH}" />
+            </geometry>
+        </visual>
+    </link>
+    <link name="front_left_link">
+        <inertial>
+            <mass value="0.01"/>
+            <origin rpy="0 0 0" xyz="0 0 0"/>
+            <inertia ixx="1e-9" ixy="0.0" ixz="0.0"
+                     iyy="1e-9" iyz="0.0"
+                     izz="1e-9"/>
+        </inertial>
+    </link>
+    <joint name="front_left_link" type="revolute">
+        <parent link="body"/>
+        <child link="front_left_link"/>
+        <origin rpy="0 0 0" xyz="${CENTER_TUBE_LENGTH/2} -${FRONT_TUBE_LENGTH/2} 0"/>
+        <axis xyz="0 0 1"/>
+        <limit effort="0" velocity="0" lower="-${PI/8}" upper="${PI/8}" />
+    </joint>
+    <link name="front_right_link">
+        <inertial>
+            <mass value="0.01"/>
+            <origin rpy="0 0 0" xyz="0 0 0"/>
+            <inertia ixx="1e-9" ixy="0.0" ixz="0.0"
+                     iyy="1e-9" iyz="0.0"
+                     izz="1e-9"/>
+        </inertial>
+    </link>
+    <joint name="front_right_link" type="revolute">
+        <parent link="body"/>
+        <child link="front_right_link"/>
+        <origin rpy="0 0 0" xyz="${CENTER_TUBE_LENGTH/2} ${FRONT_TUBE_LENGTH/2} 0"/>
+        <axis xyz="0 0 1"/>
+        <limit effort="0" velocity="0" lower="-${PI/8}" upper="${PI/8}" />
+    </joint>
+    <xacro:wheel name="front_left" origin="front_left_link" radius="0.127" x_offset="0" y_offset="0" />
+    <xacro:wheel name="front_right" origin="front_right_link" radius="0.127" x_offset="0" y_offset="0" />
+    <xacro:wheel name="back_left" origin="body" radius="0.1016" x_offset="-${CENTER_TUBE_LENGTH/2}" y_offset="-${BACK_TUBE_LENGTH/2}" />
+    <xacro:wheel name="back_right" origin="body" radius="0.1016" x_offset="-${CENTER_TUBE_LENGTH/2}" y_offset="${BACK_TUBE_LENGTH/2}" />
 </robot>

File: freehicle_description/urdf/freehicle/wheel.xacro (robot description, xacro)
@@ -1,5 +1,5 @@
 <robot name="hive" xmlns:xacro="http://www.ros.org/wiki/xacro">
-    <xacro:macro name="wheel" params="name origin dir_ns dir_ew">
-        <link name="$(arg tf_prefix)/wheel_${name}">
+    <xacro:macro name="wheel" params="name origin radius x_offset y_offset">
+        <link name="wheel_${name}">
             <inertial>
                 <mass value="1"/>
@@ -10,24 +10,21 @@
             </inertial>
             <collision name="collision">
-                <origin rpy="0 ${PI/2} 0" xyz="0 0 0"/>
+                <origin rpy="0 0 0" xyz="0 0 0"/>
                 <geometry>
-                    <cylinder radius="38e-3" length="4e-3" />
+                    <cylinder radius="${radius}" length="0.05" />
                 </geometry>
             </collision>
             <visual name="visual">
-                <origin rpy="0  0  0" xyz="0  0  0"/>
+                <origin rpy="${PI/2} 0 0" xyz="0  0  0"/>
                 <geometry>
-                    <mesh filename="package://hive_description/meshes/hive_wheel.stl" scale="1 1 ${-dir_ew * dir_ns}"/>
+                    <cylinder radius="${radius}" length="0.05" />
                 </geometry>
-                <material name="black" />
             </visual>
         </link>
-        <joint name="$(arg tf_prefix)/wheel_${name}" type="continuous">
+        <joint name="wheel_${name}" type="continuous">
             <parent link="${origin}"/>
-            <child link="$(arg tf_prefix)/wheel_${name}"/>
-            <origin rpy="0 0 0" xyz="${0.265 * dir_ew} ${0.142 * dir_ns} 0.038"/>
-            <axis xyz="-1 0 0"/>
-            <dynamics damping="${JOINT_DAMPING}" friction="${JOINT_FRICTION}" />
-            <limit effort="${MOTOR_MAX_TORQUE}" velocity="${MOTOR_MAX_VELOCITY}"/>
+            <child link="wheel_${name}"/>
+            <origin rpy="0 0 0" xyz="${x_offset} ${y_offset} 0"/>
+            <axis xyz="0 1 0"/>
         </joint>
     </xacro:macro>

Commit message: WIP camera rendering

File: freehicle_description/urdf/freehicle/freehicle.xacro (robot description, xacro)
@@ -5,4 +5,5 @@
     <xacro:property name="FRONT_TUBE_LENGTH" value="0.4826"/>
     <xacro:property name="BACK_TUBE_LENGTH" value="0.28"/>
+    <xacro:property name="WHEEL_RADIUS" value="0.1016"/>
     <xacro:property name="PI" value="3.1415926"/>
     <xacro:include filename="$(find freehicle_description)/urdf/freehicle/wheel.xacro" />
@@ -86,5 +87,5 @@
     <xacro:wheel name="front_left" origin="front_left_link" radius="0.127" x_offset="0" y_offset="0" />
     <xacro:wheel name="front_right" origin="front_right_link" radius="0.127" x_offset="0" y_offset="0" />
-    <xacro:wheel name="back_left" origin="body" radius="0.1016" x_offset="-${CENTER_TUBE_LENGTH/2}" y_offset="-${BACK_TUBE_LENGTH/2}" />
+    <xacro:wheel name="back_left" origin="body" radius="${WHEEL_RADIUS}" x_offset="-${CENTER_TUBE_LENGTH/2}" y_offset="-${BACK_TUBE_LENGTH/2}" />
     <xacro:wheel name="back_right" origin="body" radius="0.1016" x_offset="-${CENTER_TUBE_LENGTH/2}" y_offset="${BACK_TUBE_LENGTH/2}" />
 </robot>
