Commit message: WIP

File: freehicle_description/urdf/freehicle/freehicle.urdf (robot description, URDF)
Before this commit: robot hivebot, 7 links, 6 joints
Links:
- link body: mass 30 -> 1

File: freehicle_description/urdf/freehicle/freehicle.xacro (robot description, xacro)
@@ -10,9 +10,9 @@
     <link name="body">
         <inertial>
-            <mass value="30"/>
+            <mass value="1"/>
             <origin rpy="0 0 0" xyz="0 0 0"/>
-            <inertia ixx="1" ixy="0.0" ixz="0.0"
-                     iyy="1" iyz="0.0"
-                     izz="1"/>
+            <inertia ixx="0.01" ixy="0.0" ixz="0.0"
+                     iyy="0.01" iyz="0.0"
+                     izz="0.01"/>
         </inertial>
         <collision name="center_tube">

File: freehicle_description/urdf/freehicle/wheel.xacro (robot description, xacro)
@@ -10,5 +10,5 @@
             </inertial>
             <collision name="collision">
-                <origin rpy="0 0 0" xyz="0 0 0"/>
+                <origin rpy="${PI/2} 0 0" xyz="0  0  0"/>
                 <geometry>
                     <cylinder radius="${radius}" length="0.05" />

Commit message: A lot of work done

File: freehicle_description/urdf/freehicle/freehicle.urdf (robot description, URDF)
Before this commit: robot hivebot, 7 links, 6 joints
Links:
- added link camera, mass 0.01; visual cylinder length=0.03 radius=0.03
- link wheel_back_left: geometry collision cylinder length=0.01 radius=0.1016; visual cylinder length=0.01 radius=0.1016
- link wheel_back_right: geometry collision cylinder length=0.01 radius=0.1016; visual cylinder length=0.01 radius=0.1016
- link wheel_front_left: geometry collision cylinder length=0.01 radius=0.127; visual cylinder length=0.01 radius=0.127
- link wheel_front_right: geometry collision cylinder length=0.01 radius=0.127; visual cylinder length=0.01 radius=0.127
Joints:
- added joint camera: type fixed, parent body, child camera, origin xyz=0 0 0.5 rpy=0 0 0, axis 0 0 1

File: freehicle_description/urdf/freehicle/freehicle.xacro (robot description, xacro)
@@ -85,7 +85,28 @@
         <limit effort="0" velocity="0" lower="-${PI/8}" upper="${PI/8}" />
     </joint>
+    <link name="camera">
+        <inertial>
+            <mass value="0.01"/>
+            <origin rpy="0 0 0" xyz="0 0 0"/>
+            <inertia ixx="1e-9" ixy="0.0" ixz="0.0"
+                     iyy="1e-9" iyz="0.0"
+                     izz="1e-9"/>
+        </inertial>
+            <visual name="center_tube">
+            <origin rpy="0 ${PI/2} 0" xyz="0 0 0"/>
+            <geometry>
+                <cylinder radius="0.03" length="0.03" />
+            </geometry>
+        </visual>
+    </link>
+    <joint name="camera" type="fixed">
+        <parent link="body"/>
+        <child link="camera"/>
+        <origin rpy="0 0 0" xyz="0 0 0.5"/>
+        <axis xyz="0 0 1"/>
+    </joint>
     <xacro:wheel name="front_left" origin="front_left_link" radius="0.127" x_offset="0" y_offset="0" />
     <xacro:wheel name="front_right" origin="front_right_link" radius="0.127" x_offset="0" y_offset="0" />
     <xacro:wheel name="back_left" origin="body" radius="${WHEEL_RADIUS}" x_offset="-${CENTER_TUBE_LENGTH/2}" y_offset="-${BACK_TUBE_LENGTH/2}" />
-    <xacro:wheel name="back_right" origin="body" radius="0.1016" x_offset="-${CENTER_TUBE_LENGTH/2}" y_offset="${BACK_TUBE_LENGTH/2}" />
+    <xacro:wheel name="back_right" origin="body" radius="${WHEEL_RADIUS}" x_offset="-${CENTER_TUBE_LENGTH/2}" y_offset="${BACK_TUBE_LENGTH/2}" />
 </robot>

File: freehicle_description/urdf/freehicle/wheel.xacro (robot description, xacro)
@@ -12,5 +12,5 @@
                 <origin rpy="${PI/2} 0 0" xyz="0  0  0"/>
                 <geometry>
-                    <cylinder radius="${radius}" length="0.05" />
+                    <cylinder radius="${radius}" length="0.01" />
                 </geometry>
             </collision>
@@ -18,5 +18,5 @@
                 <origin rpy="${PI/2} 0 0" xyz="0  0  0"/>
                 <geometry>
-                    <cylinder radius="${radius}" length="0.05" />
+                    <cylinder radius="${radius}" length="0.01" />
                 </geometry>
             </visual>
@@ -25,4 +25,5 @@
             <parent link="${origin}"/>
             <child link="wheel_${name}"/>
+            <dynamics damping="0.0" friction="0.0"/>
             <origin rpy="0 0 0" xyz="${x_offset} ${y_offset} 0"/>
             <axis xyz="0 1 0"/>
